File: KiCad/TRAIN_MK4.kicad_pcb (KiCad board)
At the start: 2 copper layers, 80 x 57 mm, 102 parts, among them J1 Screw_Terminal_01x02, J10 Conn_01x02, J11 Conn_01x02, J2 Screw_Terminal_01x02, J3 Conn_01x02, J4 Conn_01x02, J5 Conn_01x02, J6 Conn_01x02, J7 Conn_01x02, J8 Conn_01x03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

Commit message: Update
Dividing schematic part 1
Parts:
- Q1: value SUD08P06-155L -> IPD85P04P407ATMA2

Commit message: Update
Documentation related changes and small DRU corrections
Parts:
- R6: value 20m -> 15m
Connections:
- net Net-(J8-Pin_2) renamed /FAN_PWR
- C10 pad 2: GND -> Net-(U3-V-)
- R20 pad 2: GND -> Net-(U3-V-)
- U3 pad 2: GND -> Net-(U3-V-)
Routing:
- net Net-(U3-V-): track 0.00 -> 4.61 mm
- net GND: track 4.30 -> 1.81 mm
Changed lines of the file:
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@@
 	)
 	(paper "A5")
+	(title_block
+		(title "H-PULSE-PCB")
+		(date "2025-02-24")
+		(rev "4")
+		(company "Foxhood Designs")
+	)
 	(layers
 		(0 "F.Cu" signal)
@@
 	(net 63 "Net-(SW6-B)")
 	(net 64 "unconnected-(J8-Pin_1-Pad1)")
-	(net 65 "Net-(J8-Pin_2)")
+	(net 65 "Net-(U3-V-)")
 	(net 66 "IND3")
 	(net 67 "Net-(D2-K)")
@@
 	(net 70 "unconnected-(U10-QB-Pad1)")
 	(net 71 "Net-(U1-EN)")
+	(net 72 "/FAN_PWR")
 	(footprint "TestPoint:TestPoint_Pad_2.0x2.0mm"
 		(layer "F.Cu")
@@
 		(at 87.81 77.724197)
 		(property "Reference" "U8"
-			(at -3.175 -23.495 0)
+			(at -3.175 -20.124197 0)
 			(unlocked yes)
 			(layer "F.SilkS")
@@
 				(font
 					(size 1.1684 1.1684)
-					(thickness 0.1016)
+					(thickness 0.15)
 				)
 				(justify left bottom)
@@
 			(layers "F.Cu" "F.Mask" "F.Paste")
 			(roundrect_rratio 0.212766)
-			(net 65 "Net-(J8-Pin_2)")
+			(net 72 "/FAN_PWR")
 			(pintype "passive")
 		)
@@
 			(layers "*.Cu" "*.Mask")
 			(remove_unused_layers no)
-			(net 65 "Net-(J8-Pin_2)")
+			(net 72 "/FAN_PWR")
 			(pinfunction "Pin_2")
 			(pintype "passive")
@@
 			(layers "B.Cu" "B.Mask" "B.Paste")
 			(roundrect_rratio 0.25)
-			(net 65 "Net-(J8-Pin_2)")
+			(net 72 "/FAN_PWR")
 			(pinfunction "D")
 			(pintype "passive")
@@
 			(layers "B.Cu" "B.Mask" "B.Paste")
 			(roundrect_rratio 0.25)
-			(net 1 "GND")
+			(net 65 "Net-(U3-V-)")
 			(pinfunction "V-")
 			(pintype "power_in")
@@
 			(layers "B.Cu" "B.Mask" "B.Paste")
 			(roundrect_rratio 0.208333)
-			(net 1 "GND")
+			(net 65 "Net-(U3-V-)")
 			(pintype "passive")
 		)
@@
 			(layers "B.Cu" "B.Mask" "B.Paste")
 			(roundrect_rratio 0.212766)
-			(net 1 "GND")
+			(net 65 "Net-(U3-V-)")
 			(pintype "passive")
 		)
@@
 			)
 		)
-		(property "Value" "20m"
+		(property "Value" "15m"
 			(at 0 -2.28 90)
 			(layer "B.Fab")
@@
 		(tags "DPAK TO-252 DPAK-3 TO-252-3 SOT-428")
 		(property "Reference" "Q1"
-			(at 5.056697 0.0525 0)
+			(at 5.106697 0.0525 0)
 			(layer "B.SilkS")
 			(effects
@@
 			(font
 				(size 1 1)
-				(thickness 0.1)
+				(thickness 0.15)
 			)
 			(justify left bottom)
@@
 	)
 	(segment
-		(start 110.4625 62.996697)
-		(end 111.5 61.959197)
-		(width 0.35)
-		(layer "B.Cu")
-		(net 1)
-	)
-	(segment
-		(start 109.4375 62.996697)
-		(end 110.4625 62.996697)
-		(width 0.35)
-		(layer "B.Cu")
-		(net 1)
-	)
-	(segment
 		(start 81.975 75.246697)
 		(end 81.975 76.859197)
@@
 	)
 	(segment
+		(start 101.350478 63.600478)
+		(end 102.096697 64.346697)
+		(width 0.35)
+		(layer "B.Cu")
+		(net 5)
+	)
+	(segment
 		(start 121.625 55.121697)
 		(end 120.975 55.121697)
@@
 	)
 	(segment
-		(start 101.350478 63.246697)
-		(end 102.450478 64.346697)
-		(width 0.35)
-		(layer "B.Cu")
-		(net 5)
-	)
-	(segment
 		(start 79.6 75.134197)
 		(end 79.6 75.995045)
@@
 	)
 	(segment
+		(start 105.975 64.346697)
+		(end 106.125 64.196697)
+		(width 0.35)
+		(layer "B.Cu")
+		(net 5)
+	)
+	(segment
 		(start 92.259197 73.059197)
 		(end 91.3 73.059197)
@@
 	)
 	(segment
+		(start 101.350478 63.246697)
+		(end 101.350478 63.600478)
+		(width 0.35)
+		(layer "B.Cu")
+		(net 5)
+	)
+	(segment
 		(start 89.8875 65.996697)
 		(end 89.8875 72.059197)
@@
 	)
 	(segment
-		(start 105.975 64.346697)
-		(end 106.125 64.196697)
-		(width 0.35)
-		(layer "B.Cu")
-		(net 5)
-	)
-	(segment
 		(start 74.775 84.071697)
 		(end 76.05 82.796697)
@@
 	)
 	(segment
-		(start 107.003382 65.196697)
-		(end 106.125 64.318315)
+		(start 102.096697 64.346697)
+		(end 105.975 64.346697)
 		(width 0.35)
 		(layer "B.Cu")
@@
 	)
 	(segment
-		(start 102.450478 64.346697)
-		(end 105.975 64.346697)
+		(start 107.003382 65.196697)
+		(end 106.125 64.318315)
 		(width 0.35)
 		(layer "B.Cu")
@@
 		(net 63)
 	)
-	(via
-		(at 110.1 35.534197)
-		(size 0.6)
-		(drill 0.3)
-		(layers "F.Cu" "B.Cu")
-		(net 65)
-	)
 	(segment
-		(start 107.975 35.756697)
-		(end 109.8775 35.756697)
-		(width 0.45)
+		(start 113.6 61.996697)
+		(end 111.5375 61.996697)
+		(width 0.35)
 		(layer "B.Cu")
 		(net 65)
 	)
 	(segment
-		(start 106.475 37.256697)
-		(end 106.475 42.984197)
-		(width 0.45)
+		(start 110.4625 62.996697)
+		(end 111.5 61.959197)
+		(width 0.35)
 		(layer "B.Cu")
 		(net 65)
 	)
 	(segment
-		(start 109.8775 35.756697)
-		(end 110.1 35.534197)
-		(width 0.45)
+		(start 109.4375 62.996697)
+		(end 110.4625 62.996697)
+		(width 0.35)
 		(layer "B.Cu")
 		(net 65)
 	)
-	(segment
-		(start 107.975 35.756697)
-		(end 106.475 37.256697)
-		(width 0.45)
+	(arc
+		(start 111.5375 61.996697)
+		(mid 111.510983 61.985714)
+		(end 111.5 61.959197)
+		(width 0.35)
 		(layer "B.Cu")
 		(net 65)
@@
 		(net 71)
 	)
+	(via
+		(at 110.1 35.534197)
+		(size 0.6)
+		(drill 0.3)
+		(layers "F.Cu" "B.Cu")
+		(net 72)
+	)
+	(segment
+		(start 107.975 35.756697)
+		(end 109.8775 35.756697)
+		(width 0.45)
+		(layer "B.Cu")
+		(net 72)
+	)
+	(segment
+		(start 106.475 37.256697)
+		(end 106.475 42.984197)
+		(width 0.45)
+		(layer "B.Cu")
+		(net 72)
+	)
+	(segment
+		(start 109.8775 35.756697)
+		(end 110.1 35.534197)
+		(width 0.45)
+		(layer "B.Cu")
+		(net 72)
+	)
+	(segment
+		(start 107.975 35.756697)
+		(end 106.475 37.256697)
+		(width 0.45)
+		(layer "B.Cu")
+		(net 72)
+	)
 	(zone
