File: KiCad/TRAIN_MK4.kicad_sch (KiCad schematic)
At the start: 102 parts, among them J1 Screw_Terminal_01x02, J10 Conn_01x02, J11 Conn_01x02, J2 Screw_Terminal_01x02, J3 Conn_01x02, J4 Conn_01x02, J5 Conn_01x02, J6 Conn_01x02, J7 Conn_01x02, J8 Conn_01x03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

Commit message: Update
Dividing schematic part 1
Parts:
- removed C13, C15, C18: 100n, Capacitor_SMD:C_0805_2012Metric_Pad1.18x1.45mm_HandSolder, symbol SparkFun-Capacitor:C
- removed D2: LED, LED_SMD:LED_0805_2012Metric_Pad1.15x1.40mm_HandSolder, symbol Device:LED
- removed J10, J3, J4, J5, J6, J7: Conn_01x02, Connector_JST:JST_XH_B2B-XH-A_1x02_P2.50mm_Vertical, symbol Connector_Generic:Conn_01x02
- removed J11: Conn_01x02, Connector_PinHeader_2.54mm:PinHeader_1x02_P2.54mm_Vertical_SMD_Pin1Right, symbol Connector_Generic:Conn_01x02
- removed R2: 5k, Resistor_SMD:R_0805_2012Metric_Pad1.20x1.40mm_HandSolder, symbol Device:R
- removed R22, R23, R26, R27, R28, R7: 2k, Resistor_SMD:R_0805_2012Metric_Pad1.20x1.40mm_HandSolder, symbol Device:R
- removed RN1: 10k, Resistor_SMD:R_Array_Convex_4x0603, symbol Device:R_Pack04_Split
- removed SW5, SW6: SW_SPDT, Button_Switch_THT:SW_Slide_SPDT_Straight_CK_OS102011MS2Q, symbol Switch:SW_SPDT
- removed U10: 74AHC595, Package_SO:TSSOP-16_4.4x5mm_P0.65mm, symbol 74xx:74AHC595
- removed U6: 74LVC1G240, Package_TO_SOT_SMD:SOT-23-5_HandSoldering, symbol 74xGxx:74LVC1G240
- removed U9: 74HC165, Package_SO:TSSOP-16_4.4x5mm_P0.65mm, symbol 74xx:74HC165
Connections:
- net GND: no longer C10.2, R20.2, U3.2 (V-)
- new net: C10.2, R20.2, U3.2 (V-)
Other:
- added sheet IO Expansion (SPIIO.kicad_sch)
- note removed: "IO/Expansion"
- moved on the sheet: BZ1, C1, C10, C11, C12, C14, C16, C17, C19, C2, C20, C3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

Commit message: Update
Documentation related changes and small DRU corrections
Parts:
- R6: value 20m -> 15m
Connections:
- net FAN_PWR: now reaches C14.1, J8.2 (Pin_2), Q5.3 (D)
Other:
- note added: "7-24V"
Changed lines of the file:
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@@
 		)
 	)
+	(text "7-24V"
+		(exclude_from_sim no)
+		(at 26.67 37.084 0)
+		(effects
+			(font
+				(size 1.27 1.27)
+			)
+		)
+	)
 	(text "Buzzer"
 		(exclude_from_sim no)
@@
 		)
 	)
+	(text "7-24V"
+		(exclude_from_sim no)
+		(at 112.776 38.608 0)
+		(effects
+			(font
+				(size 1.27 1.27)
+			)
+		)
+	)
 	(text "RP2040 Board"
 		(exclude_from_sim no)
@@
 		)
 	)
+	(label "FAN_PWR"
+		(at 63.5 232.41 0)
+		(effects
+			(font
+				(size 1.27 1.27)
+			)
+			(justify left bottom)
+		)
+	)
 	(global_label "TRIP"
 		(shape input)
@@
 			)
 		)
-		(property "Value" "20m"
+		(property "Value" "15m"
 			(at 99.568 39.37 90)
 			(effects
